Commit message: update

File: rsc/2dwalker.urdf (robot description, URDF)
Before this commit: robot walker, 11 links, 10 joints
Joints:
- joint left_knee: limit (none) -> lower=-0.1 upper=2.62 effort=200 velocity=28.6
- joint right_knee: limit (none) -> lower=-0.1 upper=2.62 effort=200 velocity=28.6

File: rsc/ball3D.urdf (robot description, URDF)
Before this commit: robot ball2D, 3 links, 1 joints
Links:
- link ball: geometry collision mesh filename=american_football.obj; visual mesh filename=american_football.stl
